File: hardware/demo/lora/lora.kicad_sch (KiCad schematic)
At the start: 67 parts, among them J1 BUS, J2 VIN (12 TO 16 V), J3 DEBUG, J4 SMA, J5 BUS, J6 3V3, J7 Sensor, J8 OUTPUT 1, J9 OUTPUT 2, Q1 BC847, Q2 BC847, Q3 BC847, Q4 BCP56, Q5 BC847, Q6 BSS138, Q7 BSS138, Q8 BSS84, Q9 BSS138, U1 MCP1703T-3302E/DB, U2 LoRa-E5, U3 MCP1703T-5002E/DB

Commit message: add lora pcb
Parts:
- J6: value 3V3 -> VCAP
Connections:
- net V-CAP is gone; now on net VCAP: C7.2, R11.1, R12.2, R17.1
- net +3V3: no longer J6.2 (Pin_2)
- net BUS-VCAP renamed VCAP
- net VCAP: now also J6.2 (Pin_2)
- net V-SIN renamed VSIN
- net V-SOUT renamed VSOUT
Changed lines of the file:
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@@
 	(wire
 		(pts
-			(xy 49.53 115.57) (xy 49.53 119.38)
-		)
-		(stroke
-			(width 0)
-			(type default)
-		)
-	)
-	(wire
-		(pts
 			(xy 71.12 166.37) (xy 71.12 170.18)
 		)
@@
 		)
 	)
-	(global_label "V-SIN"
+	(global_label "VSIN"
 		(shape input)
 		(at 242.57 218.44 180)
@@
 		)
 		(property "Intersheetrefs" "${INTERSHEET_REFS}"
-			(at 233.779 218.44 0)
+			(at 235.3514 218.44 0)
 			(effects
 				(font
@@
 		)
 	)
-	(global_label "V-CAP"
+	(global_label "VCAP"
 		(shape input)
 		(at 168.91 166.37 0)
@@
 		)
 		(property "Intersheetrefs" "${INTERSHEET_REFS}"
-			(at 178.1848 166.37 0)
+			(at 176.6124 166.37 0)
 			(effects
 				(font
@@
 		)
 	)
-	(global_label "V-SOUT"
+	(global_label "VSOUT"
 		(shape input)
 		(at 74.93 166.37 0)
@@
 		)
 		(property "Intersheetrefs" "${INTERSHEET_REFS}"
-			(at 85.4143 166.37 0)
+			(at 83.8419 166.37 0)
 			(effects
 				(font
@@
 		)
 	)
-	(global_label "V-CAP"
+	(global_label "VCAP"
 		(shape input)
 		(at 242.57 198.12 180)
@@
 		)
 		(property "Intersheetrefs" "${INTERSHEET_REFS}"
-			(at 233.2952 198.12 0)
+			(at 234.8676 198.12 0)
 			(effects
 				(font
@@
 		)
 	)
-	(global_label "V-SIN"
+	(global_label "VSIN"
 		(shape input)
 		(at 100.33 166.37 0)
@@
 		)
 		(property "Intersheetrefs" "${INTERSHEET_REFS}"
-			(at 109.121 166.37 0)
+			(at 107.5486 166.37 0)
 			(effects
 				(font
@@
 		)
 	)
+	(global_label "VCAP"
+		(shape input)
+		(at 49.53 119.38 0)
+		(fields_autoplaced yes)
+		(effects
+			(font
+				(size 1.27 1.27)
+			)
+			(justify left)
+		)
+		(property "Intersheetrefs" "${INTERSHEET_REFS}"
+			(at 57.2324 119.38 0)
+			(effects
+				(font
+					(size 1.27 1.27)
+				)
+				(justify left)
+				(hide yes)
+			)
+		)
+	)
 	(global_label "BOOT"
 		(shape input)
@@
 		)
 	)
-	(global_label "V-SOUT"
+	(global_label "VSOUT"
 		(shape input)
 		(at 242.57 208.28 180)
@@
 		)
 		(property "Intersheetrefs" "${INTERSHEET_REFS}"
-			(at 232.0857 208.28 0)
+			(at 233.6581 208.28 0)
 			(effects
 				(font
@@
 		)
 	)
-	(global_label "BUS-VCAP"
+	(global_label "VCAP"
 		(shape input)
 		(at 212.09 146.05 0)
@@
 		)
 		(property "Intersheetrefs" "${INTERSHEET_REFS}"
-			(at 225.1748 146.05 0)
+			(at 219.7924 146.05 0)
 			(effects
 				(font
@@
 		)
 	)
-	(global_label "BUS-VCAP"
+	(global_label "VCAP"
 		(shape input)
 		(at 242.57 86.36 0)
@@
 		)
 		(property "Intersheetrefs" "${INTERSHEET_REFS}"
-			(at 255.6548 86.36 0)
+			(at 250.2724 86.36 0)
 			(effects
 				(font
@@
 			)
 		)
-		(property "Value" "3V3"
+		(property "Value" "VCAP"
 			(at 39.37 115.57 0)
 			(effects
@@
 					(unit 1)
 				)
-			)
-		)
-	)
-	(symbol
-		(lib_id "power:+3V3")
-		(at 49.53 115.57 0)
-		(unit 1)
-		(exclude_from_sim no)
-		(in_bom yes)
-		(on_board yes)
-		(dnp no)
-		(fields_autoplaced yes)
-		(property "Reference" "#PWR014"
-			(at 49.53 119.38 0)
-			(effects
-				(font
-					(size 1.27 1.27)
-				)
-				(hide yes)
-			)
-		)
-		(property "Value" "+3V3"
-			(at 49.53 110.49 0)
-			(effects
-				(font
-					(size 1.27 1.27)
-				)
-			)
-		)
-		(property "Footprint" ""
-			(at 49.53 115.57 0)
-			(effects
-				(font
-					(size 1.27 1.27)
-				)
-				(hide yes)
-			)
-		)
-		(property "Datasheet" ""
-			(at 49.53 115.57 0)
-			(effects
-				(font
-					(size 1.27 1.27)
-				)
-				(hide yes)
-			)
-		)
-		(property "Description" "Power symbol creates a global label with name \"+3V3\""
-			(at 49.53 115.57 0)
-			(effects
-				(font
-					(size 1.27 1.27)
-				)
-				(hide yes)
-			)
-		)
-		(pin "1"
-		)
-		(instances
-			(project "lora"
-				(path "/a9584426-529a-4e0b-ae47-a85b2f3eafef"
-					(reference "#PWR014")
-					(unit 1)
-				)
